File: Hardware/USB-C to Serial.kicad_pcb (KiCad board)
At the start: 2 copper layers, 33.5 x 55 mm, 25 parts, among them IC1 ZT213LEEA, IC2 FT231XS-R, J1 5747844-4, P1 USB_C_Plug_USB2.0

Commit message: Updated files
Parts:
- added TP1: TestPoint, TestPoint:TestPoint_Pad_1.5x1.5mm, F.Cu at (164.8, 84.0)
- added TP3: TestPoint, TestPoint:TestPoint_Pad_1.5x1.5mm, F.Cu at (176.2, 84.0)
- P1: footprint SnapEDA Library:GCT_USB4155-03-C_REVA -> Expansion_Card:USB_C_Plug_Molex_105444
- moved C6 21.7 mm to (177.0, 102.5), turned to 0 degrees
- moved C7 17.6 mm to (177.0, 101.2), turned to 0 degrees
- moved C8 16.8 mm to (177.0, 100.0), turned to 0 degrees
- moved C5 12.3 mm to (173.5, 127.0), turned to 0 degrees
- moved D3 5.03 mm to (156.0, 122.2)
- moved R5 4.76 mm to (159.2, 122.2)
- moved D1 4.48 mm to (156.1, 125.2)
- moved R4 4.20 mm to (159.3, 123.8)
- moved C9 4.03 mm to (174.8, 114.5)
- moved P1 3.32 mm to (170.5, 85.0), turned to 0 degrees
- moved C3 1.40 mm to (175.8, 127.2)
- moved D2 0.15 mm to (156.0, 123.8)
Connections:
- J1 pad v-: V- -> (no net)
Routing:
- net V-: track 119.2 -> 19.2 mm, vias 10 -> 7
- net V+: track 48.5 -> 2.26 mm, vias 2 -> 0
- net Net-(D3-Pad1): track 81.5 -> 36.1 mm
- net Net-(D1-Pad1): track 68.5 -> 34.2 mm, vias 0 -> 2
- net EN: track 78.8 -> 100.0 mm, vias 6 -> 4
- net USBTXD: track 33.0 -> 45.1 mm
- net SLEEP: track 26.6 -> 38.4 mm
- net Net-(D2-Pad1): track 35.5 -> 46.7 mm, vias 0 -> 2
- net USBCTS: track 24.9 -> 16.4 mm
- net Net-(C3-Pad1): track 2.34 -> 10.1 mm
- net USBDSR: track 23.7 -> 31.0 mm
- net RTS: track 11.6 -> 18.1 mm, vias 1 -> 0
- net USBDCD: track 32.9 -> 38.8 mm
- net DTR: track 33.2 -> 27.4 mm, vias 0 -> 1
- net Net-(C1-Pad1): track 15.8 -> 21.1 mm, vias 0 -> 2
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Other:
- outline, holes or cut-outs redrawn
